File: src/mini torch with clock/light_sheet.sch (KiCad schematic (older format))
At the start: 13 parts, among them Q3 MMBTA05, Q4 MMBTA05, Q5 WST02N10, SW1 SW_Push

Commit message: clock module complete awaiting PCB
Connections:
- net at Q3.3 (C): now also R9.2
Changed lines of the file:
@@
 AR Path="/63DA6432/63DB3642" Ref="SW1"  Part="1"
 AR Path="/63DB9205/63DB3642" Ref="SW2"  Part="1"
+AR Path="/63E37469/63DB3642" Ref="SW1"  Part="1"
+AR Path="/63E38A45/63DB3642" Ref="SW2"  Part="1"
 F 0 "SW2" H 4475 4185 50  0000 C CNN
 F 1 "SW_Push" H 4475 4094 50  0000 C CNN
@@
 AR Path="/63DA6432/63DB3648" Ref="#PWR07"  Part="1"
 AR Path="/63DB9205/63DB3648" Ref="#PWR015"  Part="1"
-F 0 "#PWR015" H 7225 1650 50  0001 C CNN
+AR Path="/63E37469/63DB3648" Ref="#PWR015"  Part="1"
+AR Path="/63E38A45/63DB3648" Ref="#PWR0106"  Part="1"
+F 0 "#PWR0106" H 7225 1650 50  0001 C CNN
 F 1 "VBAT" H 7240 1973 50  0000 C CNN
 F 2 "" H 7225 1800 60  0000 C CNN
@@
 AR Path="/63DA6432/63DB364E" Ref="D3"  Part="1"
 AR Path="/63DB9205/63DB364E" Ref="D5"  Part="1"
-F 0 "D5" V 7264 1957 50  0000 R CNN
+AR Path="/63E37469/63DB364E" Ref="D3"  Part="1"
+AR Path="/63E38A45/63DB364E" Ref="D2"  Part="1"
+F 0 "D2" V 7264 1957 50  0000 R CNN
 F 1 "LED" V 7173 1957 50  0000 R CNN
 F 2 "LED_THT:LED_D3.0mm_Horizontal_O3.81mm_Z2.0mm" H 7225 2075 50  0001 C CNN
@@
 AR Path="/63DA6432/63DB3658" Ref="Q5"  Part="1"
 AR Path="/63DB9205/63DB3658" Ref="Q8"  Part="1"
-F 0 "Q8" H 7329 2721 50  0000 L CNN
+AR Path="/63E37469/63DB3658" Ref="Q5"  Part="1"
+AR Path="/63E38A45/63DB3658" Ref="Q7"  Part="1"
+F 0 "Q7" H 7329 2721 50  0000 L CNN
 F 1 "WST02N10" H 7329 2630 50  0000 L CNN
 F 2 "Package_TO_SOT_SMD:SOT-23" H 7325 2775 50  0001 C CNN
@@
 AR Path="/63DA6432/63DB365E" Ref="#PWR08"  Part="1"
 AR Path="/63DB9205/63DB365E" Ref="#PWR016"  Part="1"
-F 0 "#PWR016" H 7225 3025 50  0001 C CNN
+AR Path="/63E37469/63DB365E" Ref="#PWR016"  Part="1"
+AR Path="/63E38A45/63DB365E" Ref="#PWR0128"  Part="1"
+F 0 "#PWR0128" H 7225 3025 50  0001 C CNN
 F 1 "GND" H 7230 3102 50  0000 C CNN
 F 2 "" H 7225 3275 60  0000 C CNN
@@
 AR Path="/63DA6432/63DB3666" Ref="R13"  Part="1"
 AR Path="/63DB9205/63DB3666" Ref="R20"  Part="1"
-F 0 "R20" V 6400 2625 50  0000 L CNN
+AR Path="/63E37469/63DB3666" Ref="R13"  Part="1"
+AR Path="/63E38A45/63DB3666" Ref="R18"  Part="1"
+F 0 "R18" V 6400 2625 50  0000 L CNN
 F 1 "150R" V 6225 2575 50  0000 L CNN
 F 2 "Resistor_SMD:R_0402_1005Metric" V 6365 2665 50  0001 C CNN
@@
 AR Path="/63DA6432/63DB366D" Ref="R14"  Part="1"
 AR Path="/63DB9205/63DB366D" Ref="R21"  Part="1"
-F 0 "R21" H 6868 3071 50  0000 L CNN
+AR Path="/63E37469/63DB366D" Ref="R14"  Part="1"
+AR Path="/63E38A45/63DB366D" Ref="R19"  Part="1"
+F 0 "R19" H 6868 3071 50  0000 L CNN
 F 1 "10K" H 6868 2980 50  0000 L CNN
 F 2 "Resistor_SMD:R_0402_1005Metric" V 6840 3015 50  0001 C CNN
@@
 AR Path="/63DA6432/63DB3673" Ref="#PWR06"  Part="1"
 AR Path="/63DB9205/63DB3673" Ref="#PWR014"  Part="1"
-F 0 "#PWR014" H 6800 3000 50  0001 C CNN
+AR Path="/63E37469/63DB3673" Ref="#PWR014"  Part="1"
+AR Path="/63E38A45/63DB3673" Ref="#PWR0130"  Part="1"
+F 0 "#PWR0130" H 6800 3000 50  0001 C CNN
 F 1 "GND" H 6805 3077 50  0000 C CNN
 F 2 "" H 6800 3250 60  0000 C CNN
@@
 AR Path="/63DA6432/63DB367E" Ref="Q3"  Part="1"
 AR Path="/63DB9205/63DB367E" Ref="Q6"  Part="1"
-F 0 "Q6" H 4241 3371 50  0000 L CNN
+AR Path="/63E37469/63DB367E" Ref="Q3"  Part="1"
+AR Path="/63E38A45/63DB367E" Ref="Q2"  Part="1"
+F 0 "Q2" H 4241 3371 50  0000 L CNN
 F 1 "MMBTA05" H 4241 3280 50  0000 L CNN
 F 2 "Package_TO_SOT_SMD:SOT-23" H 4250 3425 50  0001 C CNN
@@
 AR Path="/63DA6432/63DB3684" Ref="Q4"  Part="1"
 AR Path="/63DB9205/63DB3684" Ref="Q7"  Part="1"
-F 0 "Q7" H 5615 2946 50  0000 L CNN
+AR Path="/63E37469/63DB3684" Ref="Q4"  Part="1"
+AR Path="/63E38A45/63DB3684" Ref="Q6"  Part="1"
+F 0 "Q6" H 5615 2946 50  0000 L CNN
 F 1 "MMBTA05" H 5615 2855 50  0000 L CNN
 F 2 "Package_TO_SOT_SMD:SOT-23" H 5625 3000 50  0001 C CNN
@@
 AR Path="/63DA6432/63DB368A" Ref="C10"  Part="1"
 AR Path="/63DB9205/63DB368A" Ref="C11"  Part="1"
+AR Path="/63E37469/63DB368A" Ref="C10"  Part="1"
+AR Path="/63E38A45/63DB368A" Ref="C11"  Part="1"
 F 0 "C11" H 2791 3646 50  0000 L CNN
 F 1 "10uF" H 2791 3555 50  0000 L CNN
@@
 AR Path="/63DA6432/63DB3690" Ref="R8"  Part="1"
 AR Path="/63DB9205/63DB3690" Ref="R15"  Part="1"
-F 0 "R15" H 2768 3271 50  0000 L CNN
+AR Path="/63E37469/63DB3690" Ref="R8"  Part="1"
+AR Path="/63E38A45/63DB3690" Ref="R4"  Part="1"
+F 0 "R4" H 2768 3271 50  0000 L CNN
 F 1 "1K" H 2768 3180 50  0000 L CNN
 F 2 "Resistor_SMD:R_0402_1005Metric" V 2740 3215 50  0001 C CNN
@@
 AR Path="/63DA6432/63DB3696" Ref="R9"  Part="1"
 AR Path="/63DB9205/63DB3696" Ref="R16"  Part="1"
-F 0 "R16" H 4018 2971 50  0000 L CNN
+AR Path="/63E37469/63DB3696" Ref="R9"  Part="1"
+AR Path="/63E38A45/63DB3696" Ref="R5"  Part="1"
+F 0 "R5" H 4018 2971 50  0000 L CNN
 F 1 "1K" H 4018 2880 50  0000 L CNN
 F 2 "Resistor_SMD:R_0402_1005Metric" V 3990 2915 50  0001 C CNN
@@
 AR Path="/63DA6432/63DB369C" Ref="R12"  Part="1"
 AR Path="/63DB9205/63DB369C" Ref="R19"  Part="1"
-F 0 "R19" H 5593 2421 50  0000 L CNN
+AR Path="/63E37469/63DB369C" Ref="R12"  Part="1"
+AR Path="/63E38A45/63DB369C" Ref="R17"  Part="1"
+F 0 "R17" H 5593 2421 50  0000 L CNN
 F 1 "1K" H 5593 2330 50  0000 L CNN
 F 2 "Resistor_SMD:R_0402_1005Metric" V 5565 2365 50  0001 C CNN
@@
 AR Path="/63DA6432/63DB36A2" Ref="R10"  Part="1"
 AR Path="/63DB9205/63DB36A2" Ref="R17"  Part="1"
-F 0 "R17" H 4568 3371 50  0000 L CNN
+AR Path="/63E37469/63DB36A2" Ref="R10"  Part="1"
+AR Path="/63E38A45/63DB36A2" Ref="R15"  Part="1"
+F 0 "R15" H 4568 3371 50  0000 L CNN
 F 1 "10K" H 4568 3280 50  0000 L CNN
 F 2 "Resistor_SMD:R_0402_1005Metric" V 4540 3315 50  0001 C CNN
@@
 AR Path="/63DA6432/63DB36A8" Ref="R11"  Part="1"
 AR Path="/63DB9205/63DB36A8" Ref="R18"  Part="1"
-F 0 "R18" H 5018 2946 50  0000 L CNN
+AR Path="/63E37469/63DB36A8" Ref="R11"  Part="1"
+AR Path="/63E38A45/63DB36A8" Ref="R16"  Part="1"
+F 0 "R16" H 5018 2946 50  0000 L CNN
 F 1 "10K" H 5018 2855 50  0000 L CNN
 F 2 "Resistor_SMD:R_0402_1005Metric" V 4990 2890 50  0001 C CNN
@@
 AR Path="/63DA6432/63DB36AE" Ref="#PWR04"  Part="1"
 AR Path="/63DB9205/63DB36AE" Ref="#PWR012"  Part="1"
-F 0 "#PWR012" H 5525 1850 50  0001 C CNN
+AR Path="/63E37469/63DB36AE" Ref="#PWR012"  Part="1"
+AR Path="/63E38A45/63DB36AE" Ref="#PWR0131"  Part="1"
+F 0 "#PWR0131" H 5525 1850 50  0001 C CNN
 F 1 "VBAT" H 5540 2173 50  0000 C CNN
 F 2 "" H 5525 2000 60  0000 C CNN
@@
 AR Path="/63DA6432/63DB36B5" Ref="#PWR01"  Part="1"
 AR Path="/63DB9205/63DB36B5" Ref="#PWR09"  Part="1"
-F 0 "#PWR09" H 2700 3575 50  0001 C CNN
+AR Path="/63E37469/63DB36B5" Ref="#PWR09"  Part="1"
+AR Path="/63E38A45/63DB36B5" Ref="#PWR0132"  Part="1"
+F 0 "#PWR0132" H 2700 3575 50  0001 C CNN
 F 1 "GND" H 2705 3652 50  0000 C CNN
 F 2 "" H 2700 3825 60  0000 C CNN
@@
 AR Path="/63DA6432/63DB36C2" Ref="#PWR05"  Part="1"
 AR Path="/63DB9205/63DB36C2" Ref="#PWR013"  Part="1"
-F 0 "#PWR013" H 5525 3250 50  0001 C CNN
+AR Path="/63E37469/63DB36C2" Ref="#PWR013"  Part="1"
+AR Path="/63E38A45/63DB36C2" Ref="#PWR0133"  Part="1"
+F 0 "#PWR0133" H 5525 3250 50  0001 C CNN
 F 1 "GND" H 5530 3327 50  0000 C CNN
 F 2 "" H 5525 3500 60  0000 C CNN
@@
 AR Path="/63DA6432/63DB36D7" Ref="#PWR03"  Part="1"
 AR Path="/63DB9205/63DB36D7" Ref="#PWR011"  Part="1"
-F 0 "#PWR011" H 3950 3325 50  0001 C CNN
+AR Path="/63E37469/63DB36D7" Ref="#PWR011"  Part="1"
+AR Path="/63E38A45/63DB36D7" Ref="#PWR0134"  Part="1"
+F 0 "#PWR0134" H 3950 3325 50  0001 C CNN
 F 1 "GND" H 3955 3402 50  0000 C CNN
 F 2 "" H 3950 3575 60  0000 C CNN
@@
 AR Path="/63DA6432/63DB36E0" Ref="#PWR02"  Part="1"
 AR Path="/63DB9205/63DB36E0" Ref="#PWR010"  Part="1"
-F 0 "#PWR010" H 3950 2475 50  0001 C CNN
+AR Path="/63E37469/63DB36E0" Ref="#PWR010"  Part="1"
+AR Path="/63E38A45/63DB36E0" Ref="#PWR0135"  Part="1"
+F 0 "#PWR0135" H 3950 2475 50  0001 C CNN
 F 1 "VBAT" H 3965 2798 50  0000 C CNN
 F 2 "" H 3950 2625 60  0000 C CNN
@@
 Text Notes 5950 4200 2    39   ~ 0
 QUIESENT VOLTAGE VIRTUALLY ZERO\n
+Wire Wire Line
+	3950 3075 3950 3125
 $EndSCHEMATC
